File: hardware/RevA/pcb/theadmouse.kicad_pcb (KiCad board)
At the start: 4 copper layers, 55 x 55 mm, 119 parts, among them J1 CON_SWD, J10 PJ-320D-4A, J2 CON_UART, J4 TYPE-C-31-M-12, J5 CON_BAT, J6 CON_EXT, J7 CON_EXT_RJ, J8 PJ-320D-4A, J9 PJ-320D-4A, Q1 HL2312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

Commit message: hardware: RevA: create production output for JLCPCB
These files were used to place the RevA order at JLCPCB.

Signed-off-by: Martin Pietryka <martin@pietryka.at>
Routing:
- net VDD_3V3: track 20.8 -> 18.8 mm
- net GND: vias 241 -> 242
Other:
- board text added: "Martin Pietryka, 2025 https://theadmouse.com"
- board text added: "Tina"
